File: board/cansat/Dozimetr.brd (EAGLE design)
At the start: 31.5 x 94.5 mm, 47 parts, among them U1 LMC555

Commit message: Плата дозиметра готова
Parts:
- moved R17 14.4 mm to (3.50, 82.2), turned to 180 degrees
- moved R14 12.0 mm to (10.4, 77.4), turned to 180 degrees
- moved R15 8.53 mm to (7.12, 77.4), turned to 180 degrees
- moved R11 8.31 mm to (13.7, 77.4), turned to 180 degrees
- moved R12 2.50 mm to (13.7, 75.1)
- moved R13 2.50 mm to (10.5, 75.1)
- moved R16 2.50 mm to (7.12, 75.1)
- moved DEVICE 2.06 mm to (8.33, 70.8)
- moved C5 1.50 mm to (1.91, 29.5)
- moved VR1 1.50 mm to (5.05, 64.6)
- moved R2 1.00 mm to (12.4, 50.0)
- moved SI2302-1 1.00 mm to (3.46, 85.0)
- moved D5 0.73 mm to (7.00, 34.6)
- moved R18 0.51 mm to (3.47, 79.9)
- moved D4 0.10 mm to (6.80, 38.4)
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Connections:
- removed net N$24: R17.2
- removed net N$27: R15.2
- removed net N$29: R14.2
- net N$25: now also R17.2
- net N$28: now also R15.2
- net N$30: now also R14.2
Routing:
- net GND: track 50.7 -> 152.4 mm
- net 5V1: track 45.4 -> 104.1 mm
- net N$31: track 18.5 -> 5.55 mm
- net N$4: track 43.5 -> 47.6 mm, vias 0 -> 1
- net N$19: track 53.0 -> 55.9 mm, vias 0 -> 1
- net N$30: track 2.64 -> 5.39 mm
- net N$28: track 2.53 -> 5.26 mm
- net N$2: track 10.0 -> 12.1 mm
- net DOZIMETR: track 46.5 -> 44.7 mm
- net N$6: track 14.1 -> 15.8 mm
- net N$25: track 2.63 -> 4.19 mm
- net N$8: track 51.7 -> 53.1 mm
- net BUZZER: track 8.50 -> 9.75 mm
- net N$3: track 22.0 -> 23.1 mm
- net N$9: track 3.06 -> 3.94 mm
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