File: board/cansat/Dozimetr.sch (EAGLE design)
At the start: 31 parts, among them U1 LMC555CMX/NOPB

Commit message: схема дозиметра разведена
Parts:
- added JP1: (no value), CanCubeSat:PINHD-1X2
- added JP2: (no value), pinhead:PINHD-1X5
- added JP3: (no value), pinhead:PINHD-1X4
- added R11, R14, R15, R17: 10k, rcl:R-US_R0603
- added R12, R13, R16, R18: 100R, rcl:R-US_R0603
- added S1: (no value), CanCubeSat:SWITCH-BIG
- added U$10, U$7, U$8, U$9: SI2302CDS, CanCubeSat:SI2302CDS
- R10: value 22k -> 3k3
- U$5: device CanCubeSat:RCH114NPRCH114NP -> CanCubeSat:RCH114NP
Connections:
- removed net 5V: C2.2, R10.1, U$5.1, U1.!RESET!, U1.V+
- new net 12V: S1.P
- new net 5V1: C2.2, JP1.2, R10.1, U$5.1, U1.!RESET!, U1.V+
- new net BUZZER: JP2.2, R18.2
- new net DVIG: JP2.4, R13.2
- new net GND-BUZZER: JP3.1, U$10.D
- new net GND-DVIG: JP3.3, U$8.D
- new net GND-MOTOR: JP3.2, U$9.D
- new net GND-VALVE: JP3.4, U$7.D
- new net INPUT: S1.O
- new net MOTOR: JP2.3, R16.2
- new net N$24: R17.2
- new net N$25: R18.1, U$10.G
- new net N$27: R15.2
- new net N$28: R16.1, U$9.G
- new net N$29: R14.2
- new net N$30: R13.1, U$8.G
- new net N$31: R11.2, R12.1, U$7.G
- new net VALVE: JP2.5, R12.2
- net DOZIMETR: now also JP2.1
- net GND: now also JP1.1, R11.1, R14.1, R15.1, R17.1, U$10.S, U$7.S, U$8.S, U$9.S

Commit message: Расставлены подписи на плате
Parts:
- C3: value ECAP -> 1μF
- D1, D2, D3, D4, D5: value DIODE-MBR -> MBR
- U1: value LMC555CMX/NOPB -> LMC555
- VR1: value 3362H-1-502LF -> 3362H
- renumbered JP1 to PWR, JP2 to DEVICE, JP3 to GND-DEVICE, U$10 to SI2302-1, U$6 to DOSE, U$7 to SI2302-4, U$8 to SI2302-3, U$9 to SI2302-2

Commit message: Плата дозиметра готова
Connections:
- removed net N$24: R17.2
- removed net N$27: R15.2
- removed net N$29: R14.2
- net N$25: now also R17.2
- net N$28: now also R15.2
- net N$30: now also R14.2
Changed lines of the file:
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@@
-</segment>
-</net>
-<net name="N$19" class="0">
-<segment>
-<pinref part="DOSE" gate="G$1" pin="-"/>
-<wire x1="233.68" y1="50.8" x2="228.6" y2="50.8" width="0.1524" layer="91"/>
-<pinref part="R9" gate="G$1" pin="2"/>
-<wire x1="233.68" y1="50.8" x2="248.92" y2="50.8" width="0.1524" layer="91"/>
-<junction x="233.68" y="50.8"/>
-<wire x1="248.92" y1="50.8" x2="248.92" y2="60.96" width="0.1524" layer="91"/>
-<pinref part="RT2" gate="G$1" pin="DQ"/>
-<wire x1="248.92" y1="60.96" x2="254" y2="60.96" width="0.1524" layer="91"/>
-<pinref part="C6" gate="G$1" pin="1"/>
-<wire x1="256.54" y1="60.96" x2="261.62" y2="60.96" width="0.1524" layer="91"/>
-<wire x1="279.4" y1="78.74" x2="256.54" y2="78.74" width="0.1524" layer="91"/>
-<wire x1="256.54" y1="78.74" x2="256.54" y2="60.96" width="0.1524" layer="91"/>
-<wire x1="256.54" y1="60.96" x2="254" y2="60.96" width="0.1524" layer="91"/>
 </segment>
 </net>
@@
 </segment>
 </net>
-<net name="N$24" class="0">
-<segment>
-<pinref part="R17" gate="G$1" pin="2"/>
-<wire x1="-43.18" y1="154.94" x2="-27.94" y2="154.94" width="0.1524" layer="91"/>
-</segment>
-</net>
 <net name="N$25" class="0">
 <segment>
 <pinref part="SI2302-1" gate="G$1" pin="G"/>
 <pinref part="R18" gate="G$1" pin="1"/>
-<wire x1="-27.94" y1="152.4" x2="-27.94" y2="157.48" width="0.1524" layer="91"/>
+<wire x1="-27.94" y1="152.4" x2="-27.94" y2="154.94" width="0.1524" layer="91"/>
+<pinref part="R17" gate="G$1" pin="2"/>
+<wire x1="-27.94" y1="154.94" x2="-27.94" y2="157.48" width="0.1524" layer="91"/>
+<wire x1="-43.18" y1="154.94" x2="-27.94" y2="154.94" width="0.1524" layer="91"/>
+<junction x="-27.94" y="154.94"/>
 </segment>
 </net>
@@
 </segment>
 </net>
-<net name="N$27" class="0">
-<segment>
-<pinref part="R15" gate="G$1" pin="2"/>
-<wire x1="38.1" y1="154.94" x2="53.34" y2="154.94" width="0.1524" layer="91"/>
-</segment>
-</net>
 <net name="N$28" class="0">
 <segment>
 <pinref part="SI2302-2" gate="G$1" pin="G"/>
 <pinref part="R16" gate="G$1" pin="1"/>
-<wire x1="53.34" y1="152.4" x2="53.34" y2="157.48" width="0.1524" layer="91"/>
-</segment>
-</net>
-<net name="N$29" class="0">
-<segment>
-<pinref part="R14" gate="G$1" pin="2"/>
-<wire x1="114.3" y1="154.94" x2="129.54" y2="154.94" width="0.1524" layer="91"/>
+<wire x1="53.34" y1="152.4" x2="53.34" y2="154.94" width="0.1524" layer="91"/>
+<pinref part="R15" gate="G$1" pin="2"/>
+<wire x1="53.34" y1="154.94" x2="53.34" y2="157.48" width="0.1524" layer="91"/>
+<wire x1="38.1" y1="154.94" x2="53.34" y2="154.94" width="0.1524" layer="91"/>
+<junction x="53.34" y="154.94"/>
 </segment>
 </net>
@@
 <pinref part="SI2302-3" gate="G$1" pin="G"/>
 <pinref part="R13" gate="G$1" pin="1"/>
-<wire x1="129.54" y1="152.4" x2="129.54" y2="157.48" width="0.1524" layer="91"/>
+<wire x1="129.54" y1="152.4" x2="129.54" y2="154.94" width="0.1524" layer="91"/>
+<pinref part="R14" gate="G$1" pin="2"/>
+<wire x1="129.54" y1="154.94" x2="129.54" y2="157.48" width="0.1524" layer="91"/>
+<wire x1="114.3" y1="154.94" x2="129.54" y2="154.94" width="0.1524" layer="91"/>
+<junction x="129.54" y="154.94"/>
 </segment>
 </net>
 <net name="N$31" class="0">
 <segment>
-<pinref part="R11" gate="G$1" pin="2"/>
-<wire x1="187.96" y1="154.94" x2="203.2" y2="154.94" width="0.1524" layer="91"/>
 <pinref part="SI2302-4" gate="G$1" pin="G"/>
-<wire x1="203.2" y1="152.4" x2="203.2" y2="154.94" width="0.1524" layer="91"/>
 <pinref part="R12" gate="G$1" pin="1"/>
 <wire x1="203.2" y1="160.02" x2="203.2" y2="154.94" width="0.1524" layer="91"/>
+<pinref part="R11" gate="G$1" pin="2"/>
+<wire x1="203.2" y1="154.94" x2="203.2" y2="152.4" width="0.1524" layer="91"/>
+<wire x1="187.96" y1="154.94" x2="203.2" y2="154.94" width="0.1524" layer="91"/>
 <junction x="203.2" y="154.94"/>
 </segment>
@@
 </segment>
 </net>
+<net name="N$19" class="0">
+<segment>
+<pinref part="C6" gate="G$1" pin="1"/>
+<wire x1="279.4" y1="78.74" x2="256.54" y2="78.74" width="0.1524" layer="91"/>
+<pinref part="DOSE" gate="G$1" pin="-"/>
+<wire x1="233.68" y1="50.8" x2="228.6" y2="50.8" width="0.1524" layer="91"/>
+<pinref part="R9" gate="G$1" pin="2"/>
+<wire x1="233.68" y1="50.8" x2="248.92" y2="50.8" width="0.1524" layer="91"/>
+<junction x="233.68" y="50.8"/>
+<wire x1="248.92" y1="50.8" x2="248.92" y2="60.96" width="0.1524" layer="91"/>
+<pinref part="RT2" gate="G$1" pin="DQ"/>
+<wire x1="248.92" y1="60.96" x2="256.54" y2="60.96" width="0.1524" layer="91"/>
+<wire x1="256.54" y1="60.96" x2="261.62" y2="60.96" width="0.1524" layer="91"/>
+<wire x1="256.54" y1="78.74" x2="256.54" y2="60.96" width="0.1524" layer="91"/>
+<junction x="256.54" y="60.96"/>
+</segment>
+</net>
